File: PrototypingKeyboard/PrototypingKeyboard.kicad_pcb (KiCad board)
At the start: 2 copper layers, 156 x 40 mm, 56 parts, among them J1 LEFT, J2 TOP, J3 BOTTOM, J4 RIGHT

Commit message: pictures for the lazy
Parts:
- moved J3 66.0 mm to (190.0, 165.0)
- moved J2 53.0 mm to (160.0, 95.0)
Changed lines of the file:
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@@
     (solder_mask_min_width 0.25)
     (aux_axis_origin 0 0)
-    (visible_elements FFFFFF7F)
+    (visible_elements 7FFFFFFF)
     (pcbplotparams
       (layerselection 0x010fc_ffffffff)
@@
   )
   (module Connector_PinSocket_2.54mm:PinSocket_1x13_P2.54mm_Horizontal (layer F.Cu)
-    (at 124 165 270)
+    (at 190 165 270)
     (descr "Through hole angled socket strip, 1x13, 2.54mm pitch, 8.51mm socket length, single row (from Kicad 4.0.7), script generated")
     (tags "Through hole angled socket strip THT 1x13 2.54mm single row")
@@
   )
   (module Connector_PinSocket_2.54mm:PinSocket_1x13_P2.54mm_Horizontal (layer F.Cu)
-    (at 122.5 57.5 90)
+    (at 160 95 90)
     (descr "Through hole angled socket strip, 1x13, 2.54mm pitch, 8.51mm socket length, single row (from Kicad 4.0.7), script generated")
     (tags "Through hole angled socket strip THT 1x13 2.54mm single row")
